Commit message: update

File: scout/scout_description/urdf/mini.xacro (robot description, xacro)
@@ -4,4 +4,9 @@
     <xacro:arg name="robot_namespace" default="/" />
     <xacro:arg name="urdf_extras" default="empty.urdf" />
+    <xacro:arg name="enable_ros_control" default="false" />
+    <xacro:arg name="use_skid_steer_plugin" default="true" />
+    <xacro:arg name="robot_description_param" default="robot_description" />
+    <xacro:arg name="frame_prefix" default="" />
+    <xacro:arg name="sensor_namespace" default="/" />
     <xacro:include filename="$(find scout_description)/urdf/scout_mini_wheel_1.xacro" />
     <xacro:include filename="$(find scout_description)/urdf/scout_mini_wheel_2.xacro" />
@@ -130,5 +135,5 @@
     </link>
     <joint name="laser_joint" type="fixed">
-        <origin xyz="0 0 0.23" rpy="0 0 0" />
+        <origin xyz="0 0 0.30" rpy="0 0 0" />
         <parent link="base_link" />
         <child link="laser_link" />
@@ -173,4 +178,34 @@
         <parent link="base_link" />
         <child link="camera_link" />
+    </joint>
+    <link name="imu_link">
+        <inertial>
+            <origin xyz="0.0 0.0 0.0" rpy="0 0 0" />
+            <mass value="0.01" />
+            <inertia
+                ixx="0.000001" ixy="0" ixz="0"
+                iyy="0.000001" iyz="0"
+                izz="0.000001" />
+        </inertial>
+        <visual>
+            <origin xyz="0.0 0.0 0.0" rpy="0 0 0" />
+            <geometry>
+                <box size="0.03 0.02 0.01"/>
+            </geometry>
+            <material name="imu_blue">
+                <color rgba="0.1 0.2 0.8 1.0" />
+            </material>
+        </visual>
+        <collision>
+            <origin xyz="0.0 0.0 0.0" rpy="0 0 0" />
+            <geometry>
+                <box size="0.03 0.02 0.01"/>
+            </geometry>
+        </collision>
+    </link>
+    <joint name="imu_joint" type="fixed">
+        <origin xyz="0.0 0.0 0.12" rpy="0 0 0" />
+        <parent link="base_link" />
+        <child link="imu_link" />
     </joint>
 <!--
@@ -213,5 +248,5 @@
             xyz="0 0 0"
             rpy="0 0 0" />-->
-        <origin xyz="${wheelbase/2} ${-track/2} ${wheel_vertical_offset+0.001}" rpy="1.57 0 0" />
+        <origin xyz="${wheelbase/2} ${-track/2} ${wheel_vertical_offset}" rpy="1.57 0 0" />
     </xacro:scout_mini_wheel_3>
     <xacro:scout_mini_wheel_4 wheel_prefix="rear_right" wheel_diameter="${wheel_diameter}" wheel_width="${wheel_width}">
@@ -219,5 +254,5 @@
            xyz="0 0 0"
            rpy="0 0 0" />-->
-        <origin xyz="${-wheelbase/2} ${-track/2} ${wheel_vertical_offset+0.001}" rpy="1.57 0 0" />
+        <origin xyz="${-wheelbase/2} ${-track/2} ${wheel_vertical_offset}" rpy="1.57 0 0" />
     </xacro:scout_mini_wheel_4>
     <!-- Additional definitions -->

File: scout/scout_description/urdf/scout_mini_wheel_1.xacro (robot description, xacro)
@@ -35,5 +35,5 @@
                    </inertial>
             <visual>
-                <origin xyz="0 0 0" rpy="0 0 0" />
+                <origin xyz="0 0.000996 0" rpy="0 0 0" />
                 <geometry>
                     <mesh filename="package://scout_description/meshes/wheel.dae" />
@@ -56,5 +56,5 @@
             <collision>
               <origin
-                xyz="0 0 0.03"
+                xyz="0 0 0"
                 rpy="0 0 0" />
               <geometry>
@@ -73,4 +73,5 @@
             <xacro:insert_block name="joint_pose"/>
             <axis xyz="0 0 1" rpy="0 0 0" />
+            <dynamics damping="0.1" friction="0.0" />
         </joint>
     </xacro:macro>

File: scout/scout_description/urdf/scout_mini_wheel_2.xacro (robot description, xacro)
@@ -35,5 +35,5 @@
             </inertial>
             <visual>
-                <origin xyz="0 0 0" rpy="0 0 0" />
+                <origin xyz="0 0.000996 0" rpy="0 0 0" />
                 <geometry>
                     <mesh filename="package://scout_description/meshes/wheel.dae" />
@@ -56,5 +56,5 @@
             <collision>
               <origin
-                xyz="0 0 0.03"
+                xyz="0 0 0"
                 rpy="0 0 0" />
               <geometry>
@@ -73,4 +73,5 @@
             <xacro:insert_block name="joint_pose"/>
             <axis xyz="0 0 1" rpy="0 0 0" />
+            <dynamics damping="0.1" friction="0.0" />
         </joint>
     </xacro:macro>

File: scout/scout_description/urdf/scout_mini_wheel_3.xacro (robot description, xacro)
@@ -35,5 +35,5 @@
             </inertial>
             <visual>
-                <origin xyz="0 0 0" rpy="0 0 0" />
+                <origin xyz="0 0.000996 0" rpy="0 0 0" />
                 <geometry>
                     <mesh filename="package://scout_description/meshes/wheel.dae" />
@@ -56,5 +56,5 @@
             <collision>
               <origin
-                xyz="0 0 0.03"
+                xyz="0 0 0"
                 rpy="0 0 0" />
               <geometry>
@@ -73,4 +73,5 @@
             <xacro:insert_block name="joint_pose"/>
             <axis xyz="0 0 -1" rpy="0 0 0" />
+            <dynamics damping="0.1" friction="0.0" />
         </joint>
     </xacro:macro>

File: scout/scout_description/urdf/scout_mini_wheel_4.xacro (robot description, xacro)
@@ -35,5 +35,5 @@
         </inertial>
         <visual>
-            <origin xyz="0 0 0" rpy="0 0 0" />
+            <origin xyz="0 0.000996 0" rpy="0 0 0" />
             <geometry>
                 <mesh filename="package://scout_description/meshes/wheel.dae" />
@@ -56,5 +56,5 @@
             <collision>
               <origin
-                xyz="0 0 0.03"
+                xyz="0 0 0"
                 rpy="0 0 0" />
               <geometry>
@@ -73,4 +73,5 @@
             <xacro:insert_block name="joint_pose"/>
             <axis xyz="0 0 -1" rpy="0 0 0" />
+            <dynamics damping="0.1" friction="0.0" />
         </joint>
     </xacro:macro>
