Commit message: Add an optional Helios-16 style 3D lidar to the Scout Gazebo model.
16 vertical beams, 360 deg, 10 Hz. PointCloud is converted to
PointCloud2 on /rslidar_points. The sensor stays off by default.

File: scout/urdf/mini.xacro (robot description, xacro)
@@ -10,4 +10,5 @@
     <xacro:arg name="sensor_ns" default="/" />
     <xacro:arg name="enable_lidar" default="false" />
+    <xacro:arg name="enable_rslidar" default="false" />
     <xacro:arg name="enable_camera" default="false" />
     <xacro:arg name="wheel_contact_mu2" default="0.35" />
@@ -148,4 +149,31 @@
         <parent link="base_link" />
         <child link="laser_link" />
+    </joint>
+    <link name="rslidar">
+        <inertial>
+            <origin xyz="0 0 0" rpy="0 0 0" />
+            <mass value="0.8" />
+            <inertia ixx="0.001" ixy="0" ixz="0" iyy="0.001" iyz="0" izz="0.001" />
+        </inertial>
+        <visual>
+            <origin xyz="0 0 0" rpy="0 0 0" />
+            <geometry>
+                <cylinder radius="0.05" length="0.08" />
+            </geometry>
+            <material name="helios_gray">
+                <color rgba="0.2 0.2 0.2 1" />
+            </material>
+        </visual>
+        <collision>
+            <origin xyz="0 0 0" rpy="0 0 0" />
+            <geometry>
+                <cylinder radius="0.05" length="0.08" />
+            </geometry>
+        </collision>
+    </link>
+    <joint name="rslidar_joint" type="fixed">
+        <origin xyz="0 0 0.307" rpy="0 0 0" />
+        <parent link="base_link" />
+        <child link="rslidar" />
     </joint>
  <link name="camera_link">

Commit message: scout: restore bounded wheel PI with 5ms delay and 10ms lag

File: scout/urdf/mini.xacro (robot description, xacro)
@@ -20,4 +20,6 @@
     <xacro:arg name="wheelbase" default="0.451" />
     <xacro:arg name="wheel_track" default="0.490" />
+    <xacro:arg name="wheel_effort_limit" default="3.0" />
+    <xacro:arg name="wheel_velocity_limit" default="24.0" />
     <xacro:include filename="scout_mini_wheel_1.xacro" />
     <xacro:include filename="scout_mini_wheel_2.xacro" />

File: scout/urdf/scout_mini_wheel_1.xacro (robot description, xacro)
@@ -73,4 +73,5 @@
             <xacro:insert_block name="joint_pose"/>
             <axis xyz="0 0 1" rpy="0 0 0" />
+            <limit effort="$(arg wheel_effort_limit)" velocity="$(arg wheel_velocity_limit)"/>
             <dynamics damping="0.1" friction="0.0" />
         </joint>

File: scout/urdf/scout_mini_wheel_2.xacro (robot description, xacro)
@@ -73,4 +73,5 @@
             <xacro:insert_block name="joint_pose"/>
             <axis xyz="0 0 1" rpy="0 0 0" />
+            <limit effort="$(arg wheel_effort_limit)" velocity="$(arg wheel_velocity_limit)"/>
             <dynamics damping="0.1" friction="0.0" />
         </joint>

File: scout/urdf/scout_mini_wheel_3.xacro (robot description, xacro)
@@ -73,4 +73,5 @@
             <xacro:insert_block name="joint_pose"/>
             <axis xyz="0 0 -1" rpy="0 0 0" />
+            <limit effort="$(arg wheel_effort_limit)" velocity="$(arg wheel_velocity_limit)"/>
             <dynamics damping="0.1" friction="0.0" />
         </joint>

File: scout/urdf/scout_mini_wheel_4.xacro (robot description, xacro)
@@ -73,4 +73,5 @@
             <xacro:insert_block name="joint_pose"/>
             <axis xyz="0 0 -1" rpy="0 0 0" />
+            <limit effort="$(arg wheel_effort_limit)" velocity="$(arg wheel_velocity_limit)"/>
             <dynamics damping="0.1" friction="0.0" />
         </joint>

Commit message: fix(scout): express wheel mounting rotations exactly

File: scout/urdf/mini.xacro (robot description, xacro)
@@ -277,5 +277,5 @@
             xyz="0 0 0"
             rpy="0 0 0" />-->
-        <origin xyz="${wheelbase/2} ${track/2} ${wheel_vertical_offset}" rpy="-1.57 0 0" />
+        <origin xyz="${wheelbase/2} ${track/2} ${wheel_vertical_offset}" rpy="${-pi/2} 0 0" />
     </xacro:scout_mini_wheel_1>
     <xacro:scout_mini_wheel_2 wheel_prefix="rear_left" wheel_diameter="${wheel_diameter}" wheel_width="${wheel_width}">
@@ -283,5 +283,5 @@
             xyz="0 0 0"
             rpy="0 0 0" />-->
-        <origin xyz="${-wheelbase/2} ${track/2} ${wheel_vertical_offset}" rpy="-1.57 0 0" />
+        <origin xyz="${-wheelbase/2} ${track/2} ${wheel_vertical_offset}" rpy="${-pi/2} 0 0" />
     </xacro:scout_mini_wheel_2>
     <xacro:scout_mini_wheel_3 wheel_prefix="front_right" wheel_diameter="${wheel_diameter}" wheel_width="${wheel_width}">
@@ -289,5 +289,5 @@
             xyz="0 0 0"
             rpy="0 0 0" />-->
-        <origin xyz="${wheelbase/2} ${-track/2} ${wheel_vertical_offset}" rpy="1.57 0 0" />
+        <origin xyz="${wheelbase/2} ${-track/2} ${wheel_vertical_offset}" rpy="${pi/2} 0 0" />
     </xacro:scout_mini_wheel_3>
     <xacro:scout_mini_wheel_4 wheel_prefix="rear_right" wheel_diameter="${wheel_diameter}" wheel_width="${wheel_width}">
@@ -295,5 +295,5 @@
            xyz="0 0 0"
            rpy="0 0 0" />-->
-        <origin xyz="${-wheelbase/2} ${-track/2} ${wheel_vertical_offset}" rpy="1.57 0 0" />
+        <origin xyz="${-wheelbase/2} ${-track/2} ${wheel_vertical_offset}" rpy="${pi/2} 0 0" />
     </xacro:scout_mini_wheel_4>
     <!-- Additional definitions -->

Commit message: fix(scout): align wheel collisions with retained tire geometry

File: scout/urdf/mini.xacro (robot description, xacro)
@@ -19,8 +19,10 @@
     <xacro:arg name="wheel_contact_slip2" default="0.0" />
     <xacro:arg name="wheelbase" default="0.451" />
-    <!-- Wheel mesh centers in scout_visual.urdf: y = +/-0.2082515 m. -->
+    <!-- Mounting joint separation, matching scout_visual.urdf. The retained
+         mesh's tire midpoint is offset outwards along each local wheel axis. -->
     <xacro:arg name="wheel_track" default="0.416503" />
     <xacro:arg name="wheel_effort_limit" default="3.0" />
     <xacro:arg name="wheel_velocity_limit" default="24.0" />
+    <xacro:include filename="scout_mini_wheel_collision.xacro" />
     <xacro:include filename="scout_mini_wheel_1.xacro" />
     <xacro:include filename="scout_mini_wheel_2.xacro" />

File: scout/urdf/scout_mini_wheel_1.xacro (robot description, xacro)
@@ -54,14 +54,5 @@
                 </geometry>
             </visual>
-            <collision>
-              <origin
-                xyz="0 0 0"
-                rpy="0 0 0" />
-              <geometry>
-                <!-- <mesh
-                  filename="package://scout_description/meshes/wheel.dae" /> -->
-                  <cylinder radius="0.08" length="0.084"/>
-              </geometry>
-            </collision>
+            <xacro:scout_mini_wheel_collision radius="${wheel_radius}" width="${wheel_width}"/>
         </link>
         <joint name="${wheel_prefix}_wheel" type="continuous">

File: scout/urdf/scout_mini_wheel_2.xacro (robot description, xacro)
@@ -54,14 +54,5 @@
                 </geometry>
             </visual>
-            <collision>
-              <origin
-                xyz="0 0 0"
-                rpy="0 0 0" />
-              <geometry>
-                <!-- <mesh
-                  filename="package://scout_description/meshes/wheel.dae" /> -->
-                  <cylinder radius="0.08" length="0.084"/>
-              </geometry>
-            </collision>
+            <xacro:scout_mini_wheel_collision radius="${wheel_radius}" width="${wheel_width}"/>
         </link>
         <joint name="${wheel_prefix}_wheel" type="continuous">

File: scout/urdf/scout_mini_wheel_3.xacro (robot description, xacro)
@@ -54,14 +54,5 @@
                 </geometry>
             </visual>
-            <collision>
-              <origin
-                xyz="0 0 0"
-                rpy="0 0 0" />
-              <geometry>
-                <!-- <mesh
-                  filename="package://scout_description/meshes/wheel.dae" /> -->
-                  <cylinder radius="0.08" length="0.084"/>
-              </geometry>
-            </collision>
+            <xacro:scout_mini_wheel_collision radius="${wheel_radius}" width="${wheel_width}"/>
         </link>
         <joint name="${wheel_prefix}_wheel" type="continuous">

File: scout/urdf/scout_mini_wheel_4.xacro (robot description, xacro)
@@ -54,14 +54,5 @@
             </geometry>
         </visual>
-            <collision>
-              <origin
-                xyz="0 0 0"
-                rpy="0 0 0" />
-              <geometry>
-                <!-- <mesh
-                  filename="package://scout_description/meshes/wheel.dae" /> -->
-                  <cylinder radius="0.08" length="0.084"/>
-              </geometry>
-            </collision>
+            <xacro:scout_mini_wheel_collision radius="${wheel_radius}" width="${wheel_width}"/>
         </link>
         <joint name="${wheel_prefix}_wheel" type="continuous">

Commit message: feat(visual): integrate reduced Scout assets without changing physics

File: scout/urdf/mini.xacro (robot description, xacro)
@@ -59,5 +59,5 @@
                     rpy="1.57 0 -1.57" />
             <geometry>
-                <mesh filename="package://scout_description/meshes/scout_mini_base_link2.dae" />
+                <mesh filename="package://scout_description/meshes/visual/body.dae" />
             </geometry>
         </visual>
@@ -68,5 +68,5 @@
           <geometry>
             <!-- <mesh
-              filename="package://scout_description/meshes/scout_mini_base_link2.dae" /> -->
+              filename="package://scout_description/meshes/visual/body.dae" /> -->
               <box size="0.4 0.4 0.05"/>
           </geometry>
@@ -93,9 +93,6 @@
                     rpy="0.0 0.0 3.14" />
             <geometry>
-                <mesh filename="package://scout_description/meshes/box_link.STL" />
-            </geometry>
-            <material name = "red">
-            <color rgba="1 1 1 1" />
-            </material>
+                <mesh filename="package://scout_description/meshes/visual/payload.dae" />
+            </geometry>
         </visual>
         <collision>
@@ -128,15 +125,4 @@
                 izz="0.01219" />
         </inertial>
-        <visual>
-            <origin
-                    xyz="0.0 0.0 0.0"
-                    rpy="0.0 0.0 0.0" />
-            <geometry>
-                    <cylinder radius="0.01" length="0.01"/>
-            </geometry>
-            <material name = "red">
-            <color rgba="1 1 1 1" />
-            </material>
-        </visual>
         <collision>
             <origin
@@ -159,13 +145,4 @@
             <inertia ixx="0.001" ixy="0" ixz="0" iyy="0.001" iyz="0" izz="0.001" />
         </inertial>
-        <visual>
-            <origin xyz="0 0 0" rpy="0 0 0" />
-            <geometry>
-                <cylinder radius="0.05" length="0.08" />
-            </geometry>
-            <material name="helios_gray">
-                <color rgba="0.2 0.2 0.2 1" />
-            </material>
-        </visual>
         <collision>
             <origin xyz="0 0 0" rpy="0 0 0" />
@@ -195,15 +172,4 @@
                 izz="0.01219" />
         </inertial>
-        <visual>
-            <origin
-                    xyz="0.0 0.0 0.0"
-                    rpy="0.0 0.0 0.0" />
-            <geometry>
-                    <box size="0.01 0.01 0.01"/>
-            </geometry>
-            <material name = "red">
-            <color rgba="1 1 1 1" />
-            </material>
-        </visual>
         <collision>
             <origin
@@ -229,13 +195,4 @@
                 izz="0.000001" />
         </inertial>
-        <visual>
-            <origin xyz="0.0 0.0 0.0" rpy="0 0 0" />
-            <geometry>
-                <box size="0.03 0.02 0.01"/>
-            </geometry>
-            <material name="imu_blue">
-                <color rgba="0.1 0.2 0.8 1.0" />
-            </material>
-        </visual>
         <collision>
             <origin xyz="0.0 0.0 0.0" rpy="0 0 0" />

File: scout/urdf/scout_mini_wheel_1.xacro (robot description, xacro)
@@ -37,5 +37,5 @@
                 <origin xyz="0 0.000996 0" rpy="0 0 0" />
                 <geometry>
-                    <mesh filename="package://scout_description/meshes/wheel.dae" />
+                    <mesh filename="package://scout_description/meshes/visual/wheel.dae" />
                 </geometry>
             </visual>-->
@@ -51,5 +51,5 @@
                 <origin xyz="0 0 0" rpy="0 0 0" />
                 <geometry>
-                    <mesh filename="package://scout_description/meshes/wheel.dae" />
+                    <mesh filename="package://scout_description/meshes/visual/wheel.dae" />
                 </geometry>
             </visual>
@@ -60,5 +60,5 @@
               <geometry>
                 <!-- <mesh
-                  filename="package://scout_description/meshes/wheel.dae" /> -->
+                  filename="package://scout_description/meshes/visual/wheel.dae" /> -->
                   <cylinder radius="0.08" length="0.084"/>
               </geometry>

File: scout/urdf/scout_mini_wheel_2.xacro (robot description, xacro)
@@ -37,5 +37,5 @@
                 <origin xyz="0 0.000996 0" rpy="0 0 0" />
                 <geometry>
-                    <mesh filename="package://scout_description/meshes/wheel.dae" />
+                    <mesh filename="package://scout_description/meshes/visual/wheel.dae" />
                 </geometry>
             </visual>-->
@@ -51,5 +51,5 @@
                 <origin xyz="0 0 0" rpy="0 0 0" />
                 <geometry>
-                    <mesh filename="package://scout_description/meshes/wheel.dae" />
+                    <mesh filename="package://scout_description/meshes/visual/wheel.dae" />
                 </geometry>
             </visual>
@@ -60,5 +60,5 @@
               <geometry>
                 <!-- <mesh
-                  filename="package://scout_description/meshes/wheel.dae" /> -->
+                  filename="package://scout_description/meshes/visual/wheel.dae" /> -->
                   <cylinder radius="0.08" length="0.084"/>
               </geometry>

File: scout/urdf/scout_mini_wheel_3.xacro (robot description, xacro)
@@ -37,5 +37,5 @@
                 <origin xyz="0 0.000996 0" rpy="0 0 0" />
                 <geometry>
-                    <mesh filename="package://scout_description/meshes/wheel.dae" />
+                    <mesh filename="package://scout_description/meshes/visual/wheel.dae" />
                 </geometry>
             </visual>-->
@@ -51,5 +51,5 @@
                 <origin xyz="0 0 0" rpy="0 0 0" />
                 <geometry>
-                    <mesh filename="package://scout_description/meshes/wheel.dae" />
+                    <mesh filename="package://scout_description/meshes/visual/wheel.dae" />
                 </geometry>
             </visual>
@@ -60,5 +60,5 @@
               <geometry>
                 <!-- <mesh
-                  filename="package://scout_description/meshes/wheel.dae" /> -->
+                  filename="package://scout_description/meshes/visual/wheel.dae" /> -->
                   <cylinder radius="0.08" length="0.084"/>
               </geometry>

File: scout/urdf/scout_mini_wheel_4.xacro (robot description, xacro)
@@ -37,5 +37,5 @@
             <origin xyz="0 0.000996 0" rpy="0 0 0" />
             <geometry>
-                <mesh filename="package://scout_description/meshes/wheel.dae" />
+                <mesh filename="package://scout_description/meshes/visual/wheel.dae" />
             </geometry>
         </visual>-->
@@ -51,5 +51,5 @@
             <origin xyz="0 0 0" rpy="0 0 0" />
             <geometry>
-                <mesh filename="package://scout_description/meshes/wheel.dae" />
+                <mesh filename="package://scout_description/meshes/visual/wheel.dae" />
             </geometry>
         </visual>
@@ -60,5 +60,5 @@
               <geometry>
                 <!-- <mesh
-                  filename="package://scout_description/meshes/wheel.dae" /> -->
+                  filename="package://scout_description/meshes/visual/wheel.dae" /> -->
                   <cylinder radius="0.08" length="0.084"/>
               </geometry>

Commit message: fix(scout): propagate physical wheel radius and derive coherent wheel inertias

File: scout/urdf/mini.xacro (robot description, xacro)
@@ -22,7 +22,13 @@
          mesh's tire midpoint is offset outwards along each local wheel axis. -->
     <xacro:arg name="wheel_track" default="0.416503" />
+    <xacro:arg name="wheel_radius" default="0.08" />
+    <xacro:arg name="wheel_mass" default="3.0" />
+    <xacro:arg name="wheel_width" default="0.084" />
+    <xacro:arg name="wheel_joint_damping" default="0.1" />
+    <xacro:arg name="wheel_inertial_axial_offset" default="0.0" />
     <xacro:arg name="wheel_effort_limit" default="3.0" />
     <xacro:arg name="wheel_velocity_limit" default="24.0" />
     <xacro:include filename="scout_mini_wheel_collision.xacro" />
+    <xacro:include filename="scout_mini_wheel_inertial.xacro" />
     <xacro:include filename="scout_mini_wheel_1.xacro" />
     <xacro:include filename="scout_mini_wheel_2.xacro" />
@@ -38,11 +44,10 @@
     <xacro:property name="track" value="$(arg wheel_track)"/>
     <xacro:property name="wheel_vertical_offset" value="-0.100998" />
-    <xacro:property name="wheel_diameter" value="0.16" />
-    <xacro:property name="wheel_width" value="0.084" />
+    <xacro:property name="wheel_diameter" value="${2.0 * float('$(arg wheel_radius)')}" />
+    <xacro:property name="wheel_width" value="${float('$(arg wheel_width)')}" />
 <!--    <xacro:property name="track" value="0.3426" />
     <xacro:property name="wheelbase" value="0.3181"/>
     <xacro:property name="wheel_vertical_offset" value="-0.160000047342231" />-->
-    <xacro:property name="wheel_length" value="0.8e-01" />
-    <xacro:property name="wheel_radius" value="1.600e-01" />
+    <!-- Wheel radius is a physical parameter shared with command allocation. -->
     <!-- Base link -->
     <link name="base_link">

File: scout/urdf/scout_mini_wheel_1.xacro (robot description, xacro)
@@ -40,12 +40,5 @@
                 </geometry>
             </visual>-->
-            <inertial>
-                <mass value="3" />
-                <origin xyz="0 0 0" />
-                <inertia
-                    ixx="0.006564" ixy="0" ixz="0"
-                    iyy="0.006564" iyz="0"
-                    izz="0.0096"/>
-              </inertial>
+            <xacro:scout_mini_wheel_inertial radius="${wheel_radius}" width="${wheel_width}"/>
             <visual>
                 <origin xyz="0 0 0" rpy="0 0 0" />
@@ -65,5 +58,5 @@
             <axis xyz="0 0 1" rpy="0 0 0" />
             <limit effort="$(arg wheel_effort_limit)" velocity="$(arg wheel_velocity_limit)"/>
-            <dynamics damping="0.1" friction="0.0" />
+            <dynamics damping="$(arg wheel_joint_damping)" friction="0.0" />
         </joint>
     </xacro:macro>

File: scout/urdf/scout_mini_wheel_2.xacro (robot description, xacro)
@@ -40,12 +40,5 @@
                 </geometry>
             </visual>-->
-            <inertial>
-                <mass value="3" />
-                <origin xyz="0 0 0" />
-                <inertia
-                    ixx="0.006564" ixy="0" ixz="0"
-                    iyy="0.006564" iyz="0"
-                    izz="0.0096"/>
-              </inertial>
+            <xacro:scout_mini_wheel_inertial radius="${wheel_radius}" width="${wheel_width}"/>
             <visual>
                 <origin xyz="0 0 0" rpy="0 0 0" />
@@ -65,5 +58,5 @@
             <axis xyz="0 0 1" rpy="0 0 0" />
             <limit effort="$(arg wheel_effort_limit)" velocity="$(arg wheel_velocity_limit)"/>
-            <dynamics damping="0.1" friction="0.0" />
+            <dynamics damping="$(arg wheel_joint_damping)" friction="0.0" />
         </joint>
     </xacro:macro>

File: scout/urdf/scout_mini_wheel_3.xacro (robot description, xacro)
@@ -40,12 +40,5 @@
                 </geometry>
             </visual>-->
-            <inertial>
-                <mass value="3" />
-                <origin xyz="0 0 0" />
-                <inertia
-                    ixx="0.006564" ixy="0" ixz="0"
-                    iyy="0.006564" iyz="0"
-                    izz="0.0096"/>
-              </inertial>
+            <xacro:scout_mini_wheel_inertial radius="${wheel_radius}" width="${wheel_width}"/>
             <visual>
                 <origin xyz="0 0 0" rpy="0 0 0" />
@@ -65,5 +58,5 @@
             <axis xyz="0 0 -1" rpy="0 0 0" />
             <limit effort="$(arg wheel_effort_limit)" velocity="$(arg wheel_velocity_limit)"/>
-            <dynamics damping="0.1" friction="0.0" />
+            <dynamics damping="$(arg wheel_joint_damping)" friction="0.0" />
         </joint>
     </xacro:macro>

File: scout/urdf/scout_mini_wheel_4.xacro (robot description, xacro)
@@ -40,12 +40,5 @@
             </geometry>
         </visual>-->
-        <inertial>
-            <mass value="3" />
-            <origin xyz="0 0 0" />
-                <inertia
-                    ixx="0.006564" ixy="0" ixz="0"
-                    iyy="0.006564" iyz="0"
-                    izz="0.0096"/>
-              </inertial>
+        <xacro:scout_mini_wheel_inertial radius="${wheel_radius}" width="${wheel_width}"/>
         <visual>
             <origin xyz="0 0 0" rpy="0 0 0" />
@@ -65,5 +58,5 @@
             <axis xyz="0 0 -1" rpy="0 0 0" />
             <limit effort="$(arg wheel_effort_limit)" velocity="$(arg wheel_velocity_limit)"/>
-            <dynamics damping="0.1" friction="0.0" />
+            <dynamics damping="$(arg wheel_joint_damping)" friction="0.0" />
         </joint>
     </xacro:macro>

Commit message: Fix Scout block-laser projection and expose sensor parameters

File: scout/urdf/mini.xacro (robot description, xacro)
@@ -10,4 +10,12 @@
     <xacro:arg name="enable_lidar" default="false" />
     <xacro:arg name="enable_rslidar" default="false" />
+    <xacro:arg name="rslidar_rate_hz" default="10" />
+    <xacro:arg name="rslidar_min_range_meters" default="0.2" />
+    <xacro:arg name="rslidar_range_meters" default="80.0" />
+    <xacro:arg name="rslidar_hfov_deg" default="0" />
+    <xacro:arg name="rslidar_vfov_deg" default="0" />
+    <xacro:arg name="rslidar_hres" default="900" />
+    <xacro:arg name="rslidar_vres" default="16" />
+    <xacro:arg name="rslidar_pose" default="0 0 0.307 0 0 0" />
     <xacro:arg name="enable_camera" default="false" />
     <xacro:arg name="enable_simple_lidar" default="false" />
@@ -169,5 +177,5 @@
     </link>
     <joint name="rslidar_joint" type="fixed">
-        <origin xyz="0 0 0.307" rpy="0 0 0" />
+        <origin xyz="${' '.join('$(arg rslidar_pose)'.split()[:3])}" rpy="${' '.join('$(arg rslidar_pose)'.split()[3:])}" />
         <parent link="base_link" />
         <child link="rslidar" />
